Commit message: vehicle UI

File: src/vehicle/sample_vehicle_launch/sample_vehicle_description/urdf/vehicle.xacro (robot description, xacro)
@@ -6,7 +6,7 @@
   <link name="base_link">
     <visual>
-      <origin xyz="${vehicle_info['/**']['ros__parameters']['wheel_base']/2.0} 0 0" rpy="${pi/2.0} 0 ${pi}"/>
+      <origin xyz="${vehicle_info['/**']['ros__parameters']['wheel_base']/2.0} 0 0" rpy="${pi/2.0} 0 ${pi/2.0}"/>
       <geometry>
-        <mesh filename="package://sample_vehicle_description/mesh/lexus.dae" scale="1 1 1"/>
+        <mesh filename="package://sample_vehicle_description/mesh/IONIQ5.dae" scale="1 1 1"/>
       </geometry>
     </visual>
